File: adafruit_feather_main_board/adafruit_feather_template.kicad_pcb (KiCad board)
At the start: 2 copper layers, 50.8 x 22.9 mm, 24 parts, among them J1 4045_Connector_PH_2pos_RA_SMD, J2 4039_Header_Male_Vert_16pin_0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, J3 3096_USBC_RA_SMD, J4 4040_Header_Male_Vert_12pin_0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, Q1 4043_DMG3414_Nch_Mosfet_SOT23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, SW1 RST, U1 4042_MCP73831_Battery_Charger, U2 3093_MIC5225_3v3, U3 CRG, U4 4044_LED_RED_SMD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

Commit message: Added template icon and info file
Parts:
- removed R10: 4008_Resistor_SMD_10k_0.125W_1%, Shulltronics_Generics:RES-0402
- added G***: LOGO, Shulltronics_Generics:LOGO-feather, B.Cu at (154.3, 93.0)
- added REF**: Shulltronics_Logo, Shulltronics_Generics:Shulltronics_Logo, B.Cu at (170.2, 86.0)
- U4: value 4044_LED_RED_SMD -> STAT
- moved C2 29.4 mm to (141.4, 100.1), turned to 180 degrees
- moved U1 25.4 mm to (145.0, 93.2), turned to -90 degrees
- moved U2 21.2 mm to (141.4, 97.7), turned to 180 degrees
- moved R1 20.8 mm to (131.4, 69.8)
- moved R6 20.6 mm to (147.3, 93.2), turned to 90 degrees
- moved C3 20.4 mm to (142.6, 93.2), turned to -90 degrees
- moved SW1 19.8 mm to (122.5, 97.6)
- moved R4 18.4 mm to (140.2, 91.2)
- moved R9 16.2 mm to (135.7, 84.6)
- moved C1 13.9 mm to (148.6, 85.0)
- moved U5 13.8 mm to (133.3, 84.6)
- moved R7 1.21 mm to (135.7, 98.5)
- moved R5 1.16 mm to (140.2, 94.2)
- moved R3 1.16 mm to (140.2, 92.2), turned to 180 degrees
- moved U3 1.15 mm to (133.3, 98.5)
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Connections:
- net Net-(R6-Pad1) renamed /PROG
- net Net-(R7-Pad1) renamed /STAT
Other:
- copper layers 2 -> 4
