File: adafruit_feather_main_board/adafruit_feather_template.kicad_sch (KiCad schematic)
At the start: 24 parts, among them J1 4045_Connector_PH_2pos_RA_SMD, J2 4039_Header_Male_Vert_16pin_0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, J3 3096_USBC_RA_SMD, J4 4040_Header_Male_Vert_12pin_0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, Q1 4043_DMG3414_Nch_Mosfet_SOT23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, SW1 RST, U1 4042_MCP73831_Battery_Charger, U2 3093_MIC5225_3v3, U3 CRG, U4 4044_LED_RED_SMD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

Commit message: Added template icon and info file
Parts:
- removed R10: 4008_Resistor_SMD_10k_0.125W_1%, Shulltronics_Generics:RES-0402, symbol Shulltronics_Passives:4008_Resistor_SMD_10k_0.125W_1%
- U4: value 4044_LED_RED_SMD -> STAT
Connections:
- net STAT: now reaches R7.1, U1.1 (STAT)
- net PROG: now reaches R6.1, U1.5 (PROG)
Changed lines of the file:
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@@
     (effects (font (size 1.27 1.27)) (justify left bottom))
+  )
+  (label "PROG" (at 55.88 35.56 180)
+    (effects (font (size 1.27 1.27)) (justify right bottom))
   )
   (label "SCL" (at 70.612 191.262 0)
@@
   (label "~{RST}" (at 48.514 155.702 180)
     (effects (font (size 1.27 1.27)) (justify right bottom))
+  )
+  (label "STAT" (at 78.74 35.56 0)
+    (effects (font (size 1.27 1.27)) (justify left bottom))
   )
   (label "CC2" (at 41.275 114.3 0)
@@
   )
   (symbol (lib_id "Shulltronics_Opto:4044_LED_RED_SMD") (at 91.44 116.205 270) (unit 1)
-    (in_bom yes) (on_board yes) (fields_autoplaced)
+    (in_bom yes) (on_board yes)
     (property "Reference" "U4" (id 0) (at 97.155 114.8079 90)
       (effects (font (size 1.27 1.27)) (justify left))
     )
-    (property "Value" "4044_LED_RED_SMD" (id 1) (at 82.55 116.205 0)
-      (effects (font (size 1.27 1.27)) hide)
-    )
+    (property "Value" "STAT" (id 1) (at 99.06 119.38 90))
     (property "Footprint" "Shulltronics_Generics:LED_0402" (id 2) (at 77.47 116.205 0)
       (effects (font (size 1.27 1.27)) hide)
@@
     )
     (property "SPN" "4036" (id 4) (at 92.075 70.485 90)
-      (effects (font (size 1.27 1.27)) (justify left))
-    )
-    (pin "1")
-    (pin "2")
-  )
-  (symbol (lib_id "Shulltronics_Passives:4008_Resistor_SMD_10k_0.125W_1%") (at 144.78 85.09 0) (unit 1)
-    (in_bom yes) (on_board yes)
-    (property "Reference" "R10" (id 0) (at 147.32 85.09 0)
-      (effects (font (size 1.27 1.27)) (justify left))
-    )
-    (property "Value" "4008_Resistor_SMD_10k_0.125W_1%" (id 1) (at 149.86 78.74 90)
-      (effects (font (size 1.27 1.27)) hide)
-    )
-    (property "Footprint" "Shulltronics_Generics:RES-0402" (id 2) (at 144.78 105.41 0)
-      (effects (font (size 1.27 1.27)) hide)
-    )
-    (property "Datasheet" "https://www.te.com/commerce/DocumentDelivery/DDEController?Action=srchrtrv&DocNm=9-1773463-9&DocType=DS&DocLang=English" (id 3) (at 146.05 101.6 0)
-      (effects (font (size 1.27 1.27)) hide)
-    )
-    (property "SPN" "4008" (id 4) (at 138.43 85.09 0)
-      (effects (font (size 1.27 1.27)) hide)
-    )
-    (property "Val" "10k" (id 5) (at 144.78 86.995 90)
       (effects (font (size 1.27 1.27)) (justify left))
     )
@@
       (reference "R9") (unit 1) (value "4038_Resistor_SMD_100_0.125W_1%") (footprint "Shulltronics_Generics:RES-0402")
     )
-    (path "/347e83a7-ef7f-4ef7-b610-d71da01b71a2"
-      (reference "R10") (unit 1) (value "4008_Resistor_SMD_10k_0.125W_1%") (footprint "Shulltronics_Generics:RES-0402")
-    )
     (path "/3fdeaed2-7e2a-4286-8c32-55164331f861"
       (reference "SW1") (unit 1) (value "RST") (footprint "Shulltronics_ElectroMechanical:4012_PushButton_NO_SMD")
@@
     )
     (path "/13692434-9c3c-402f-8ce4-9ffbfd0334d9"
-      (reference "U4") (unit 1) (value "4044_LED_RED_SMD") (footprint "Shulltronics_Generics:LED_0402")
+      (reference "U4") (unit 1) (value "STAT") (footprint "Shulltronics_Generics:LED_0402")
     )
     (path "/32cf9bd7-7bc9-4ff7-9da1-e3fc3874f42d"
